File: KiCad/Power_Brick/Power_Brick.kicad_pcb (KiCad board)
At the start: 2 copper layers, 38 parts, among them J1 Conn_01x06, J2 Conn_01x09, J3 MKDS5_2-9_5_6pos_PowerPad, Q1 CSD18540Q5B, Q2 CSD18540Q5B, Q3 CSD18540Q5B, Q4 CSD18540Q5B, Q5 CSD18540Q5B, Q6 CSD18540Q5B, Q7 CSD18540Q5B, Q8 CSD18540Q5B, SW1 SMD_5.2x5.2mm_h1.9mm, U1 DRV8704DCPR, U2 ADS1220xPW, U3 ADS1220xPW

Commit message: Beta Design
Parts:
- added C12: 10nF, PCM_SparkFun-Capacitor:C_0402_1005Metric, F.Cu at (197.4, 153.2)
- added C13: 10nF, PCM_SparkFun-Capacitor:C_0402_1005Metric, F.Cu at (194.4, 153.2)
- added C14: 10nF, PCM_SparkFun-Capacitor:C_0402_1005Metric, F.Cu at (202.4, 148.7)
- added C15: 10nF, PCM_SparkFun-Capacitor:C_0402_1005Metric, F.Cu at (202.4, 151.7)
- added C16: 10nF, PCM_SparkFun-Capacitor:C_0402_1005Metric, F.Cu at (189.6, 151.7)
- added C17: 10nF, PCM_SparkFun-Capacitor:C_0402_1005Metric, F.Cu at (189.6, 148.7)
- added C18: 0.1uF, PCM_SparkFun-Capacitor:C_0402_1005Metric, F.Cu at (200.9, 150.2)
- added C19: 0.1uF, PCM_SparkFun-Capacitor:C_0402_1005Metric, F.Cu at (191.1, 150.2)
- added C20: 0.1uF, PCM_SparkFun-Capacitor:C_0402_1005Metric, F.Cu at (195.9, 151.7)
- added C21: 0.1uF, PCM_SparkFun-Capacitor:C_0402_1005Metric, F.Cu at (202.4, 145.9)
- added C22: 0.1uF, PCM_SparkFun-Capacitor:C_0402_1005Metric, F.Cu at (202.4, 147.5)
- added C23: 10nF, PCM_SparkFun-Capacitor:C_0402_1005Metric, F.Cu at (232.3, 153.1)
- added C24: 10nF, PCM_SparkFun-Capacitor:C_0402_1005Metric, F.Cu at (229.3, 153.1)
- added C25: 10nF, PCM_SparkFun-Capacitor:C_0402_1005Metric, F.Cu at (237.3, 148.6)
- added C26: 10nF, PCM_SparkFun-Capacitor:C_0402_1005Metric, F.Cu at (237.3, 151.6)
- added C27: 10nF, PCM_SparkFun-Capacitor:C_0402_1005Metric, F.Cu at (224.6, 151.6)
- added C28: 10nF, PCM_SparkFun-Capacitor:C_0402_1005Metric, F.Cu at (224.6, 148.6)
- added C29: 0.1uF, PCM_SparkFun-Capacitor:C_0402_1005Metric, F.Cu at (235.8, 150.1)
- added C30: 0.1uF, PCM_SparkFun-Capacitor:C_0402_1005Metric, F.Cu at (226.1, 150.1)
- added C31: 0.1uF, PCM_SparkFun-Capacitor:C_0402_1005Metric, F.Cu at (230.8, 151.6)
- added C32: 0.1uF, PCM_SparkFun-Capacitor:C_0402_1005Metric, F.Cu at (237.3, 145.9)
- added C33: 0.1uF, PCM_SparkFun-Capacitor:C_0402_1005Metric, F.Cu at (237.4, 147.5)
- added H1: MountingHole, MountingHole:MountingHole_3.2mm_M3, F.Cu at (243.8, 94.4)
- added H2: MountingHole, MountingHole:MountingHole_3.2mm_M3, F.Cu at (181.2, 94.4)
- added H3: MountingHole, MountingHole:MountingHole_3.2mm_M3, F.Cu at (181.2, 156.9)
- added H4: MountingHole, MountingHole:MountingHole_3.2mm_M3, F.Cu at (243.8, 156.9)
- added J4: MKDS5_2-9_5_1pos_PowerPad, Power_Brick:MKDS5_2-9_5_1pos_PowerPad, F.Cu at (242.5, 103.1)
- added J5: MKDS5_2-9_5_4pos_PowerPad, Power_Brick:MKDS5_2-9_5_4pos_PowerPad, F.Cu at (213.0, 97.0)
- added J6: Conn_01x04, Connector_PinHeader_2.54mm:PinHeader_1x04_P2.54mm_Vertical, F.Cu at (188.1, 158.9)
- added J7: Conn_01x04, Connector_PinHeader_2.54mm:PinHeader_1x04_P2.54mm_Vertical, F.Cu at (229.8, 158.9)
- added JP1: Jumper_2_Bridged, PCM_SparkFun-Jumper:Jumper_2_NO, F.Cu at (204.6, 150.2)
- added JP2: Jumper_2_Bridged, PCM_SparkFun-Jumper:Jumper_2_NO, F.Cu at (187.4, 150.2)
- added JP3: Jumper_2_Bridged, PCM_SparkFun-Jumper:Jumper_2_NO, F.Cu at (187.4, 147.8)
- added JP4: Jumper_2_Bridged, PCM_SparkFun-Jumper:Jumper_2_NO, F.Cu at (239.8, 150.2)
- added JP5: Jumper_2_Bridged, PCM_SparkFun-Jumper:Jumper_2_NO, F.Cu at (222.3, 150.1)
- added JP6: Jumper_2_Bridged, PCM_SparkFun-Jumper:Jumper_2_NO, F.Cu at (222.3, 147.6)
- added NT1: NetTie_2, Power_Brick:NetTie-2_SMD_Pad0.25mm, F.Cu at (194.5, 112.9)
- added NT2: NetTie_2, Power_Brick:NetTie-2_SMD_Pad0.25mm, F.Cu at (206.0, 113.1)
- added NT3: NetTie_2, Power_Brick:NetTie-2_SMD_Pad0.25mm, F.Cu at (219.0, 113.4)
- added NT4: NetTie_2, Power_Brick:NetTie-2_SMD_Pad0.25mm, F.Cu at (230.5, 113.1)
- added NT5: NetTie_2, Power_Brick:NetTie-2_SMD_Pad0.25mm, F.Cu at (191.9, 156.9)
- added NT6: NetTie_2, Power_Brick:NetTie-2_SMD_Pad0.25mm, F.Cu at (233.5, 156.6)
- added NT7: NetTie_2, NetTie:NetTie-2_SMD_Pad2.0mm, F.Cu at (204.2, 156.9)
- added NT8: NetTie_2, NetTie:NetTie-2_SMD_Pad0.5mm, F.Cu at (188.5, 139.9)
- added NT9: NetTie_2, NetTie:NetTie-2_SMD_Pad0.5mm, F.Cu at (243.8, 139.6)
- added R10: 20k, PCM_SparkFun-Resistor:R_0402_1005Metric, F.Cu at (195.9, 154.7)
- added R11: 0, PCM_SparkFun-Resistor:R_0402_1005Metric, F.Cu at (196.4, 153.2)
- added R12: 10k, PCM_SparkFun-Resistor:R_0402_1005Metric, F.Cu at (195.4, 153.2)
- added R13: 10k, PCM_SparkFun-Resistor:R_0402_1005Metric, F.Cu at (202.4, 149.7)
- added R14: 10k, PCM_SparkFun-Resistor:R_0402_1005Metric, F.Cu at (202.4, 150.7)
- added R15: 10k, PCM_SparkFun-Resistor:R_0402_1005Metric, F.Cu at (189.6, 150.7)
- added R16: 10k, PCM_SparkFun-Resistor:R_0402_1005Metric, F.Cu at (189.6, 149.7)
- added R17: 22, PCM_SparkFun-Resistor:R_0402_1005Metric, F.Cu at (193.1, 144.4)
- added R18: 22, PCM_SparkFun-Resistor:R_0402_1005Metric, F.Cu at (198.9, 144.4)
- added R19: 22, PCM_SparkFun-Resistor:R_0402_1005Metric, F.Cu at (199.9, 144.4)
- added R20: 22, PCM_SparkFun-Resistor:R_0402_1005Metric, F.Cu at (192.1, 144.4)
- added R21: 22, PCM_SparkFun-Resistor:R_0402_1005Metric, F.Cu at (200.9, 144.4)
- added R22: 20k, PCM_SparkFun-Resistor:R_0402_1005Metric, F.Cu at (230.8, 154.6)
- added R23: 0, PCM_SparkFun-Resistor:R_0402_1005Metric, F.Cu at (231.3, 153.1)
- added R24: 10k, PCM_SparkFun-Resistor:R_0402_1005Metric, F.Cu at (230.3, 153.1)
- added R25: 10k, PCM_SparkFun-Resistor:R_0402_1005Metric, F.Cu at (237.3, 149.6)
- added R26: 10k, PCM_SparkFun-Resistor:R_0402_1005Metric, F.Cu at (237.3, 150.6)
- added R27: 10k, PCM_SparkFun-Resistor:R_0402_1005Metric, F.Cu at (224.6, 150.6)
- added R28: 10k, PCM_SparkFun-Resistor:R_0402_1005Metric, F.Cu at (224.6, 149.6)
- added R29: 22, PCM_SparkFun-Resistor:R_0402_1005Metric, F.Cu at (228.1, 144.4)
- added R30: 22, PCM_SparkFun-Resistor:R_0402_1005Metric, F.Cu at (233.8, 144.4)
- added R31: 22, PCM_SparkFun-Resistor:R_0402_1005Metric, F.Cu at (234.8, 144.4)
- added R32: 22, PCM_SparkFun-Resistor:R_0402_1005Metric, F.Cu at (227.1, 144.4)
- added R33: 22, PCM_SparkFun-Resistor:R_0402_1005Metric, F.Cu at (235.8, 144.4)
- J1: value Conn_01x06 -> Conn_01x10; footprint Connector_PinHeader_2.54mm:PinHeader_1x06_P2.54mm_Vertical -> Connector_PinHeader_2.54mm:PinHeader_1x10_P2.54mm_Vertical
- J3: value MKDS5_2-9_5_6pos_PowerPad -> MKDS5_2-9_5_1pos_PowerPad; footprint Power_Brick:MKDS5_2-9_5_6pos_PowerPad -> Power_Brick:MKDS5_2-9_5_1pos_PowerPad
- moved U3 110.0 mm to (231.0, 148.4)
- moved C6 101.1 mm to (186.2, 118.1)
- moved C7 100.7 mm to (186.2, 132.6)
- moved J1 98.5 mm to (201.7, 158.9), turned to 90 degrees
- moved C9 93.7 mm to (238.8, 118.1)
- moved C10 93.3 mm to (238.8, 132.6)
- moved U1 92.3 mm to (212.5, 122.6)
- moved R4 91.7 mm to (197.7, 118.6)
- moved Q6 91.1 mm to (221.8, 109.6)
- moved Q7 91.1 mm to (233.8, 107.1)
- moved Q8 91.1 mm to (227.8, 109.6)
- moved Q1 90.8 mm to (191.2, 107.1)
- moved Q2 90.8 mm to (197.2, 109.6)
- moved Q3 90.8 mm to (209.2, 107.1)
- moved Q4 90.8 mm to (203.2, 109.6)
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Connections:
- D1 pad 1: Net-(D1-K) -> /FAULT_N
- D3 pad 1: Net-(D3-K) -> /SLEEP_N_IN
- J1 pad 1: VCC -> +3.3V
- J1 pad 2: GND -> GNDD
- J1 pad 3: /SDI -> /SCLK
- J1 pad 4: /SDO -> /SDI
- J1 pad 5: /SCLK -> /SDO
- J2 pad 1: /AIN1 -> +3.3V
- J2 pad 2: /AIN2 -> GND
- J2 pad 3: /BIN1 -> /SLEEP_N_IN
- J2 pad 4: /BIN2 -> /RESET
- J2 pad 5: /RESET -> /FAULT_N
- J2 pad 6: /SLEEP_N -> /AIN1
- J2 pad 7: /FAULT -> /AIN2
- J2 pad 8: VCC -> /BIN1
- J2 pad 9: GND -> /BIN2
- J3 pad 1: /AOUT1 -> VBUS
- Q1 pad 1: /AOUT1 -> /MA1
- Q1 pad 2: /AOUT1 -> /MA1
- Q1 pad 3: /AOUT1 -> /MA1
- Q2 pad 1: /SENSE_A -> /AISENP
- Q2 pad 2: /SENSE_A -> /AISENP
- Q2 pad 3: /SENSE_A -> /AISENP
- Q2 pad 5_6_7_8: /AOUT1 -> /MA1
- Q3 pad 1: /AOUT2 -> /MA2
- Q3 pad 2: /AOUT2 -> /MA2
- Q3 pad 3: /AOUT2 -> /MA2
- Q4 pad 1: /SENSE_A -> /AISENP
- Q4 pad 2: /SENSE_A -> /AISENP
- Q4 pad 3: /SENSE_A -> /AISENP
- Q4 pad 5_6_7_8: /AOUT2 -> /MA2
- Q5 pad 1: /BOUT1 -> /MB1
- Q5 pad 2: /BOUT1 -> /MB1
- Q5 pad 3: /BOUT1 -> /MB1
- Q6 pad 1: /SENS_B -> /BISENP
- Q6 pad 2: /SENS_B -> /BISENP
- Q6 pad 3: /SENS_B -> /BISENP
- Q6 pad 5_6_7_8: /BOUT1 -> /MB1
- Q7 pad 1: /BOUT2 -> /MB2
- Q7 pad 2: /BOUT2 -> /MB2
- Q7 pad 3: /BOUT2 -> /MB2
- Q8 pad 1: /SENS_B -> /BISENP
- Q8 pad 2: /SENS_B -> /BISENP
- Q8 pad 3: /SENS_B -> /BISENP
- Q8 pad 5_6_7_8: /BOUT2 -> /MB2
- R1 pad 2: VCC -> +3.3V
- R2 pad 1: VCC -> +3.3V
- R2 pad 2: Net-(D1-K) -> /FAULT_N
- R4 pad 2: /SENSE_A -> /AISENP
- R5 pad 1: Net-(D3-K) -> /SLEEP_N_IN
- R6 pad 2: Net-(D3-K) -> /SLEEP_N_IN
- R7 pad 1: Net-(D3-K) -> /SLEEP_N_IN
- R8 pad 1: VCC -> +3.3V
- R9 pad 2: /SENS_B -> /BISENP
- SW1 pad 1: VCC -> +3.3V
- U1 pad 18: Net-(D1-K) -> /FAULT_N
- U1 pad 24: /BISENN -> GND
- U1 pad 33: /AISENN -> GND
- U2 pad 1: unconnected-(U2-SCLK-Pad1) -> Net-(U2-SCLK)
- U2 pad 10: unconnected-(U2-AIN1-Pad10) -> Net-(U2-AIN1)
- U2 pad 11: unconnected-(U2-AIN0/REFP1-Pad11) -> Net-(U2-AIN0/REFP1)
- U2 pad 12: unconnected-(U2-AVDD-Pad12) -> +3.3V
- U2 pad 13: unconnected-(U2-DVDD-Pad13) -> +3.3V
- U2 pad 14: unconnected-(U2-~{DRDY}-Pad14) -> Net-(U2-~{DRDY})
- U2 pad 15: unconnected-(U2-DOUT/~{DRDY}-Pad15) -> Net-(U2-DOUT/~{DRDY})
- U2 pad 16: unconnected-(U2-DIN-Pad16) -> Net-(U2-DIN)
- U2 pad 2: unconnected-(U2-~{CS}-Pad2) -> Net-(U2-~{CS})
- U2 pad 3: unconnected-(U2-CLK-Pad3) -> GNDD
- U2 pad 4: unconnected-(U2-DGND-Pad4) -> GNDD
- U2 pad 5: unconnected-(U2-AVSS-Pad5) -> GNDA
- U2 pad 6: unconnected-(U2-AIN3/REFN1-Pad6) -> Net-(U2-AIN3/REFN1)
- U2 pad 7: unconnected-(U2-AIN2-Pad7) -> Net-(U2-AIN2)
- U2 pad 8: unconnected-(U2-REFN0-Pad8) -> Net-(U2-REFN0)
- U2 pad 9: unconnected-(U2-REFP0-Pad9) -> Net-(U2-REFP0)
- U3 pad 1: unconnected-(U3-SCLK-Pad1) -> Net-(U3-SCLK)
- U3 pad 10: unconnected-(U3-AIN1-Pad10) -> Net-(U3-AIN1)
- U3 pad 11: unconnected-(U3-AIN0/REFP1-Pad11) -> Net-(U3-AIN0/REFP1)
- U3 pad 12: unconnected-(U3-AVDD-Pad12) -> +3.3V
- U3 pad 13: unconnected-(U3-DVDD-Pad13) -> +3.3V
- U3 pad 14: unconnected-(U3-~{DRDY}-Pad14) -> Net-(U3-~{DRDY})
- U3 pad 15: unconnected-(U3-DOUT/~{DRDY}-Pad15) -> Net-(U3-DOUT/~{DRDY})
- U3 pad 16: unconnected-(U3-DIN-Pad16) -> Net-(U3-DIN)
- U3 pad 2: unconnected-(U3-~{CS}-Pad2) -> Net-(U3-~{CS})
- U3 pad 3: unconnected-(U3-CLK-Pad3) -> GNDD
- U3 pad 4: unconnected-(U3-DGND-Pad4) -> GNDD
- U3 pad 5: unconnected-(U3-AVSS-Pad5) -> GNDA
- U3 pad 6: unconnected-(U3-AIN3/REFN1-Pad6) -> Net-(U3-AIN3/REFN1)
- U3 pad 7: unconnected-(U3-AIN2-Pad7) -> Net-(U3-AIN2)
- U3 pad 8: unconnected-(U3-REFN0-Pad8) -> Net-(U3-REFN0)
- U3 pad 9: unconnected-(U3-REFP0-Pad9) -> Net-(U3-REFP0)
Routing:
- net +3.3V: track 0.00 -> 162.3 mm, vias 0 -> 5
- net /SCLK: track 0.00 -> 77.9 mm, vias 0 -> 6
- net /SDI: track 0.00 -> 76.2 mm, vias 0 -> 6
- net /SDO: track 0.00 -> 75.8 mm, vias 0 -> 4
- net /CS_T1: track 0.00 -> 45.2 mm, vias 0 -> 2
- net /SCS: track 0.00 -> 44.7 mm, vias 0 -> 2
- net /DRDY_N_T2: track 0.00 -> 42.4 mm, vias 0 -> 2
- net GND: track 0.00 -> 39.1 mm, vias 0 -> 99
- net /DRDY_N_T1: track 0.00 -> 33.9 mm
- net /A1HS: track 0.87 -> 32.3 mm, vias 0 -> 2
- net /RESET: track 0.00 -> 31.4 mm, vias 0 -> 3
- net GNDA: track 0.00 -> 30.9 mm, vias 0 -> 29
- net VBUS: track 7.00 -> 36.4 mm, vias 0 -> 73
- net /FAULT_N: track 0.00 -> 28.9 mm, vias 0 -> 1
- net /CS_T2: track 0.00 -> 28.3 mm, vias 0 -> 2
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- added copper zone on F.Cu, net /AISENP
- added copper zone on F.Cu, net /BISENP
- added copper zone on F.Cu, net /MA1
- added copper zone on F.Cu, net /MA2
- added copper zone on F.Cu, net /MB1
- added copper zone on F.Cu, net /MB2
- added copper zone on B.Cu, net GND
- added copper zone on F.Cu, net GND
- added copper zone on B.Cu, net GNDA
- added copper zone on F.Cu, net GNDA
- added copper zone on B.Cu, net GNDD
- added copper zone on F.Cu, net GNDD
- added copper zone on B.Cu, net VBUS
- added copper zone on F.Cu, net VBUS
Other:
- board outline added: 70 x 70 mm

Commit message: KiCad beta
Routing:
- net VBUS: vias 73 -> 88
Changed lines of the file:
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@@
 	)
 	(via
-		(at 208.5 112.85625)
+		(at 215.132267 111.312021)
+		(size 0.6)
+		(drill 0.3)
+		(layers "F.Cu" "B.Cu")
+		(free yes)
+		(net 4)
+	)
+	(via
+		(at 208.25 112)
+		(size 0.6)
+		(drill 0.3)
+		(layers "F.Cu" "B.Cu")
+		(free yes)
+		(net 4)
+	)
+	(via
+		(at 214.632267 112.062021)
 		(size 0.6)
 		(drill 0.3)
@@
 	)
 	(via
+		(at 214.132267 111.312021)
+		(size 0.6)
+		(drill 0.3)
+		(layers "F.Cu" "B.Cu")
+		(free yes)
+		(net 4)
+	)
+	(via
 		(at 237.25 111.85625)
 		(size 0.6)
@@
 	)
 	(via
-		(at 209.25 111.35625)
+		(at 208.75 111.35625)
 		(size 0.6)
 		(drill 0.3)
@@
 	)
 	(via
-		(at 212.5 107.85625)
+		(at 212.5 107.39375)
 		(size 0.6)
 		(drill 0.3)
@@
 	)
 	(via
+		(at 217.132267 112.705771)
+		(size 0.6)
+		(drill 0.3)
+		(layers "F.Cu" "B.Cu")
+		(free yes)
+		(net 4)
+	)
+	(via
+		(at 214.132267 112.705771)
+		(size 0.6)
+		(drill 0.3)
+		(layers "F.Cu" "B.Cu")
+		(free yes)
+		(net 4)
+	)
+	(via
 		(at 193.25 113.85625)
 		(size 0.6)
@@
 	)
 	(via
-		(at 216.5 112.85625)
-		(size 0.6)
-		(drill 0.3)
-		(layers "F.Cu" "B.Cu")
-		(free yes)
-		(net 4)
-	)
-	(via
 		(at 204.75 127.60625)
 		(size 0.6)
@@
 	)
 	(via
-		(at 215.5 111.35625)
-		(size 0.6)
-		(drill 0.3)
-		(layers "F.Cu" "B.Cu")
-		(free yes)
-		(net 4)
-	)
-	(via
 		(at 237.25 115.85625)
 		(size 0.6)
@@
 	)
 	(via
-		(at 212.5 109.60625)
+		(at 212.5 110.39375)
+		(size 0.6)
+		(drill 0.3)
+		(layers "F.Cu" "B.Cu")
+		(free yes)
+		(net 4)
+	)
+	(via
+		(at 212.5 109.39375)
 		(size 0.6)
 		(drill 0.3)
@@
 	)
 	(via
+		(at 215.632267 112.062021)
+		(size 0.6)
+		(drill 0.3)
+		(layers "F.Cu" "B.Cu")
+		(free yes)
+		(net 4)
+	)
+	(via
 		(at 234.75 115.85625)
 		(size 0.6)
@@
 	)
 	(via
-		(at 217 111.35625)
-		(size 0.6)
-		(drill 0.3)
-		(layers "F.Cu" "B.Cu")
-		(free yes)
-		(net 4)
-	)
-	(via
 		(at 237.25 119.60625)
 		(size 0.6)
@@
 	)
 	(via
+		(at 209.75 112.75)
+		(size 0.6)
+		(drill 0.3)
+		(layers "F.Cu" "B.Cu")
+		(free yes)
+		(net 4)
+	)
+	(via
 		(at 237.25 131.10625)
 		(size 0.6)
@@
 	)
 	(via
-		(at 212.5 106.60625)
-		(size 0.6)
-		(drill 0.3)
-		(layers "F.Cu" "B.Cu")
-		(free yes)
-		(net 4)
-	)
-	(via
-		(at 214 111.35625)
-		(size 0.6)
-		(drill 0.3)
-		(layers "F.Cu" "B.Cu")
-		(free yes)
-		(net 4)
-	)
-	(via
-		(at 210.25 112.85625)
+		(at 212.5 106.5)
+		(size 0.6)
+		(drill 0.3)
+		(layers "F.Cu" "B.Cu")
+		(free yes)
+		(net 4)
+	)
+	(via
+		(at 210.75 111.35625)
+		(size 0.6)
+		(drill 0.3)
+		(layers "F.Cu" "B.Cu")
+		(free yes)
+		(net 4)
+	)
+	(via
+		(at 209.25 112)
 		(size 0.6)
 		(drill 0.3)
@@
 	)
 	(via
+		(at 207.75 112.75)
+		(size 0.6)
+		(drill 0.3)
+		(layers "F.Cu" "B.Cu")
+		(free yes)
+		(net 4)
+	)
+	(via
+		(at 216.132267 111.312021)
+		(size 0.6)
+		(drill 0.3)
+		(layers "F.Cu" "B.Cu")
+		(free yes)
+		(net 4)
+	)
+	(via
 		(at 193.25 126.60625)
 		(size 0.6)
@@
 	)
 	(via
-		(at 214.75 112.85625)
+		(at 208.75 112.75)
+		(size 0.6)
+		(drill 0.3)
+		(layers "F.Cu" "B.Cu")
+		(free yes)
+		(net 4)
+	)
+	(via
+		(at 216.132267 112.705771)
 		(size 0.6)
 		(drill 0.3)
@@
 	)
 	(via
-		(at 211.75 112.85625)
+		(at 215.132267 112.705771)
+		(size 0.6)
+		(drill 0.3)
+		(layers "F.Cu" "B.Cu")
+		(free yes)
+		(net 4)
+	)
+	(via
+		(at 217.132267 111.312021)
+		(size 0.6)
+		(drill 0.3)
+		(layers "F.Cu" "B.Cu")
+		(free yes)
+		(net 4)
+	)
+	(via
+		(at 212.5 112.75)
+		(size 0.6)
+		(drill 0.3)
+		(layers "F.Cu" "B.Cu")
+		(free yes)
+		(net 4)
+	)
+	(via
+		(at 210.25 112)
 		(size 0.6)
 		(drill 0.3)
@@
 	)
 	(via
+		(at 212.5 108.39375)
+		(size 0.6)
+		(drill 0.3)
+		(layers "F.Cu" "B.Cu")
+		(free yes)
+		(net 4)
+	)
+	(via
 		(at 231.75 119.60625)
 		(size 0.6)
@@
 	)
 	(via
-		(at 213.25 112.85625)
+		(at 211.25 112)
 		(size 0.6)
 		(drill 0.3)
@@
 	)
 	(via
+		(at 210.75 112.75)
+		(size 0.6)
+		(drill 0.3)
+		(layers "F.Cu" "B.Cu")
+		(free yes)
+		(net 4)
+	)
+	(via
 		(at 190.25 113.85625)
 		(size 0.6)
@@
 	)
 	(via
-		(at 211 111.35625)
+		(at 209.75 111.35625)
 		(size 0.6)
 		(drill 0.3)
@@
 	)
 	(via
+		(at 216.632267 112.062021)
+		(size 0.6)
+		(drill 0.3)
+		(layers "F.Cu" "B.Cu")
+		(free yes)
+		(net 4)
+	)
+	(via
 		(at 234.75 119.60625)
 		(size 0.6)
@@
 		(size 0.6)
 		(drill 0.3)
+		(layers "F.Cu" "B.Cu")
+		(free yes)
+		(net 4)
+	)
+	(via
+		(at 213.632267 112.062021)
+		(size 0.6)
+		(drill 0.3)

Commit message: KiCad beta
Routing:
- net GND: vias 99 -> 139
