File: KiCad/Power_Brick/Power_Brick/Power_Brick.kicad_sch (KiCad schematic)
At the start: 109 parts, among them J1 Conn_01x10, J2 Conn_01x09, J3 MKDS5_2-9_5_1pos_PowerPad, J4 MKDS5_2-9_5_1pos_PowerPad, J5 MKDS5_2-9_5_4pos_PowerPad, J6 Conn_01x04, J7 Conn_01x04, Q1 CSD18540Q5B, Q2 CSD18540Q5B, Q3 CSD18540Q5B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

Commit message: KiCad beta
Parts:
- SW1: footprint PCM_SparkFun-Switch:Push_SMD_5.2x5.2mm_h1.9mm -> PCM_SparkFun-Switch:Push_SMD_4.6x2.8mm_h1.9mm; symbol PCM_SparkFun-Switch:SPST_Push_SMD_5.2x5.2mm_h1.9mm -> PCM_SparkFun-Switch:SPST_Push_SMD_4.6x2.8mm_h1.9mm; PROD_ID SWCH-08247 -> SWCH-13065
Changed lines of the file:
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@@
 	)
 	(symbol
-		(lib_id "PCM_SparkFun-Switch:SPST_Push_SMD_5.2x5.2mm_h1.9mm")
+		(lib_id "PCM_SparkFun-Switch:SPST_Push_SMD_4.6x2.8mm_h1.9mm")
 		(at 104.14 171.45 0)
 		(unit 1)
@@
 			)
 		)
-		(property "Footprint" "PCM_SparkFun-Switch:Push_SMD_5.2x5.2mm_h1.9mm"
+		(property "Footprint" "PCM_SparkFun-Switch:Push_SMD_4.6x2.8mm_h1.9mm"
 			(at 104.14 176.53 0)
 			(effects
@@
 			)
 		)
-		(property "Datasheet" "https://sten-eswitch-13110800-production.s3.amazonaws.com/system/asset/product_line/data_sheet/165/TL3342.pdf"
+		(property "Datasheet" "https://www.ckswitches.com/media/1479/kmr2.pdf"
 			(at 104.14 181.61 0)
 			(effects
@@
 			)
 		)
-		(property "PROD_ID" "SWCH-08247"
+		(property "PROD_ID" "SWCH-13065"
 			(at 104.14 179.07 0)
 			(effects
 				(font
+					(size 1.27 1.27)
+				)
+				(hide yes)
+			)
+		)
+		(property "Mfg Part#" ""
+			(at 104.14 171.45 0)
+			(effects
+				(font

Commit message: Revised fault and capacitor ratings
Parts:
- removed D3: Zener, Diode_SMD:D_SOD-323_HandSoldering, symbol PCM_SparkFun-DiscreteSemi:D_Zener
- removed R5: 100k, PCM_SparkFun-Resistor:R_0402_1005Metric, symbol PCM_SparkFun-Resistor:100k_0402
- C5: Voltage 50V -> 100V
- R7: value 22 -> 330
Connections:
- net SLEEP_N: now also R6.2, R7.1; no longer R7.2
- net SLEEP_N_IN: now also R7.2; no longer R6.2, R7.1
Other:
- moved on the sheet: R7

Commit message: Digital Grount Updates
Connections:
- net GND: no longer J2.2 (Pin_2)
- net GNDD: now also J2.2 (Pin_2)
Changed lines of the file:
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@@
 			)
 		)
-		(property "Value" "GND"
+		(property "Value" "GNDD"
 			(at 69.85 234.95 0)
 			(do_not_autoplace yes)
